File: VolumeControl.kicad_pcb (KiCad board)
At the start: 2 copper layers, 66.5 x 52.1 mm, 42 parts, among them J1 Input R/GND/L, J2 SPI, J3 Screw_Terminal_01x03, J4 5V Supply, J5 Lout, J6 Rout, J7 SubOut, U1 AD5290, U2 AD5290, U3 TL082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

Commit message: Fixed DRC errors fine adjusted some positions Nice Silkscreen Gerber files exported
Parts:
- C1, C10, C2, C5, C6: value C_Polarized 10µF 50V -> 10µF 50V
- moved R12 1.08 mm to (55.0, 36.2)
- moved R13 1.07 mm to (51.2, 26.0)
- moved J4 0.97 mm to (27.9, 27.9)
- moved J2 0.96 mm to (27.9, 40.6)
- moved J1 0.44 mm to (33.0, 50.8)
Routing:
- net Net-(C2-Pad1): track 10.1 -> 8.17 mm
- net Net-(J3-Pad3): track 19.7 -> 21.2 mm
- net Net-(J3-Pad1): track 25.7 -> 26.6 mm
- net -12VA: track 131.1 -> 132.1 mm
- net +5V: track 14.1 -> 15.0 mm
- net /CS1: track 51.7 -> 52.5 mm
- net /SDI: track 40.8 -> 41.6 mm
- net /CLK: track 51.2 -> 52.0 mm
- net +12VA: track 113.7 -> 114.5 mm
Other:
- board text added: "10uF 50V: C1,2,5,6,10 100nF: C3,4,9,11,12,13"
